File: Schematic/GenMemBlock.kicad_pcb (KiCad board)
At the start: 4 copper layers, 99.6 x 75.6 mm, 40 parts, among them J1 MCU_HEADER, J2 ADDR_BUS, J3 DATA_BUS, J4 CART_A20, J5 CART_B10, J6 CART_B20, J7 CART_A10, J8 SDCARD, P1 MD-CART-FINGERS-doragasu, U1 74HCT595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

Commit message: moved to single board with SPI splitter
Parts:
- added R4: 10K, Resistor_SMD:R_0805_2012Metric_Pad1.20x1.40mm_HandSolder, B.Cu at (112.9, 93.5)
- J8: value SDCARD -> Conn_01x07_Female
Connections:
- C11 pad 1: Net-(C11-Pad1) -> +5V
Routing:
- net SPI_MISO_FB_OE#: track 14.6 -> 17.3 mm
- net +5V: track 563.7 -> 566.0 mm, vias 41 -> 42
- net SPI_CLK: track 23.6 -> 22.8 mm
